File: hw/teacup-carrier.kicad_sch (KiCad schematic)
At the start: 128 parts, among them J1 AH58893-T9B10-3F, J2 TYPE-C-31-M-12, J20 HDR_J20, J21 HDR_J21, J22 HDR_J22, J23 HDR_J23, J24 HDR_J24, J25 HDR_J25, J26 HDR_J26, J27 HDR_J27, J28 HDR_J28, J29 HDR_J29, J3 TE_292303-7, J30 HDR_J30, J31 HDR_J31, J32 HDR_J32, J33 HDR_J33, J34 HDR_J34, J35 HDR_J35, J4 Hirose_DM3D-SF, J5 Wuerth_694106301002, J6 AudioJack4_Ground, J7 SFW15R-2STE1LF, J8 SFW15R-2STE1LF, J9 TYPE-C-31-M-12, Q1 AO3401A, Q2 AO3401A, SW1 SSSS711403, SW2 SSSS711403, U1 AP62600SJ-7, U10 TS5A3166, U11 DIP-8 Socket, U12 TPS2053BDR, U13 W25Q32JVSS, U14 TPS22990DMLR, U15 TCA9555PWR, U2 AP62300WU-7, U3 MCP4661-104E_ST, U4 TPS22990DMLR, U5 AZ1117CH-3.3TRG1, U6 AZ1117CH-1.8TRG1, U7 AP62300WU-7, U8 ESP32-S3-WROOM-1-N16R2, U9 TS5A3166

Commit message: Convert large pin-breakout headers to double-row, J1-ordered pinout
J20/J21/J25/J27/J30-J35 now use Conn_02xNN_Odd_Even + PinHeader_2xNN
footprints instead of single-row 1xNN -- half the physical length, and
KiCad's odd/even pin numbering keeps each header's signals in the same
J1-sequential order they were already assigned, just zig-zagged across
two columns instead of one long row. Odd GND+signal counts get a 2nd
GND appended at the far pin to fill the row evenly. J22-J24/J26/J28/J29
(<=5 pins) stay single-row.

Regenerated headers.kicad_sch/teacup-carrier.kicad_sch/CONNECTIONS.txt
via the existing schgen toolchain: 0 overlaps, ERC violation set
unchanged from baseline (429, byte-identical). Rebuilt
teacup-carrier.kicad_pcb via build_pcb.py for the new footprints --
rough cluster placement only, no routing.
Parts:
- removed J20: HDR_J20, Connector_PinHeader_2.54mm:PinHeader_1x11_P2.54mm_Vertical, symbol Connector_Generic:Conn_01x11
- removed J21: HDR_J21, Connector_PinHeader_2.54mm:PinHeader_1x11_P2.54mm_Vertical, symbol Connector_Generic:Conn_01x11
- removed J25: HDR_J25, Connector_PinHeader_2.54mm:PinHeader_1x07_P2.54mm_Vertical, symbol Connector_Generic:Conn_01x07
- removed J27: HDR_J27, Connector_PinHeader_2.54mm:PinHeader_1x09_P2.54mm_Vertical, symbol Connector_Generic:Conn_01x09
- removed J30: HDR_J30, Connector_PinHeader_2.54mm:PinHeader_1x17_P2.54mm_Vertical, symbol Connector_Generic:Conn_01x17
- removed J31: HDR_J31, Connector_PinHeader_2.54mm:PinHeader_1x24_P2.54mm_Vertical, symbol Connector_Generic:Conn_01x24
- removed J32: HDR_J32, Connector_PinHeader_2.54mm:PinHeader_1x25_P2.54mm_Vertical, symbol Connector_Generic:Conn_01x25
- removed J33: HDR_J33, Connector_PinHeader_2.54mm:PinHeader_1x25_P2.54mm_Vertical, symbol Connector_Generic:Conn_01x25
- removed J34: HDR_J34, Connector_PinHeader_2.54mm:PinHeader_1x25_P2.54mm_Vertical, symbol Connector_Generic:Conn_01x25
- removed J35: HDR_J35, Connector_PinHeader_2.54mm:PinHeader_1x25_P2.54mm_Vertical, symbol Connector_Generic:Conn_01x25
- added J20: HDR_J20, Connector_PinHeader_2.54mm:PinHeader_2x06_P2.54mm_Vertical, symbol Connector_Generic:Conn_02x06_Odd_Even
- added J21: HDR_J21, Connector_PinHeader_2.54mm:PinHeader_2x06_P2.54mm_Vertical, symbol Connector_Generic:Conn_02x06_Odd_Even
- added J25: HDR_J25, Connector_PinHeader_2.54mm:PinHeader_2x04_P2.54mm_Vertical, symbol Connector_Generic:Conn_02x04_Odd_Even
- added J27: HDR_J27, Connector_PinHeader_2.54mm:PinHeader_2x05_P2.54mm_Vertical, symbol Connector_Generic:Conn_02x05_Odd_Even
- added J30: HDR_J30, Connector_PinHeader_2.54mm:PinHeader_2x09_P2.54mm_Vertical, symbol Connector_Generic:Conn_02x09_Odd_Even
- added J31: HDR_J31, Connector_PinHeader_2.54mm:PinHeader_2x12_P2.54mm_Vertical, symbol Connector_Generic:Conn_02x12_Odd_Even
- added J32: HDR_J32, Connector_PinHeader_2.54mm:PinHeader_2x13_P2.54mm_Vertical, symbol Connector_Generic:Conn_02x13_Odd_Even
- added J33: HDR_J33, Connector_PinHeader_2.54mm:PinHeader_2x13_P2.54mm_Vertical, symbol Connector_Generic:Conn_02x13_Odd_Even
- added J34: HDR_J34, Connector_PinHeader_2.54mm:PinHeader_2x13_P2.54mm_Vertical, symbol Connector_Generic:Conn_02x13_Odd_Even
- added J35: HDR_J35, Connector_PinHeader_2.54mm:PinHeader_2x13_P2.54mm_Vertical, symbol Connector_Generic:Conn_02x13_Odd_Even
Connections:
- net GMAC0_MDCK: now also J20.3 (Pin_3)
- net GMAC0_MDIO: now also J20.2 (Pin_2)
- net GMAC0_PHYCLK: now also J20.5 (Pin_5)
- net GMAC0_RXD0: now also J20.10 (Pin_10)
- net GMAC0_RXD1: now also J20.11 (Pin_11)
- net GMAC0_RXDV: now also J20.9 (Pin_9)
- net GMAC0_TXCLK: now also J20.4 (Pin_4)
- net GMAC0_TXD0: now also J20.7 (Pin_7)
- net GMAC0_TXD1: now also J20.8 (Pin_8)
- net GMAC0_TXEN: now also J20.6 (Pin_6)
- net GMAC1_MDCK: now also J21.3 (Pin_3)
- net GMAC1_MDIO: now also J21.2 (Pin_2)
- net GMAC1_PHYCLK: now also J21.5 (Pin_5)
- net GMAC1_RXD0: now also J21.10 (Pin_10)
- net GMAC1_RXD1: now also J21.11 (Pin_11)
- net GMAC1_RXDV: now also J21.9 (Pin_9)
- net GMAC1_TXCLK: now also J21.4 (Pin_4)
- net GMAC1_TXD0: now also J21.7 (Pin_7)
- net GMAC1_TXD1: now also J21.8 (Pin_8)
- net GMAC1_TXEN: now also J21.6 (Pin_6)
- net GND: now also J20.1 (Pin_1), J20.12 (Pin_12), J21.1 (Pin_1), J21.12 (Pin_12), J25.1 (Pin_1), J25.8 (Pin_8), J27.1 (Pin_1), J27.10 (Pin_10), J30.1 (Pin_1), J30.18 (Pin_18), J31.1 (Pin_1), J32.1 (Pin_1), J32.26 (Pin_26), J33.1 (Pin_1), J33.26 (Pin_26), J34.1 (Pin_1), J34.26 (Pin_26), J35.1 (Pin_1), J35.26 (Pin_26)
- net GPIO0: now also J30.2 (Pin_2)
- net GPIO1: now also J30.3 (Pin_3)
- net GPIO10: now also J30.12 (Pin_12)
- net GPIO11: now also J30.13 (Pin_13)
- net GPIO12: now also J30.14 (Pin_14)
- net GPIO13: now also J30.15 (Pin_15)
- net GPIO14: now also J30.16 (Pin_16)
- net GPIO15: now also J30.17 (Pin_17)
- net GPIO2: now also J30.4 (Pin_4)
- net GPIO3: now also J30.5 (Pin_5)
- net GPIO4: now also J30.6 (Pin_6)
- net GPIO5: now also J30.7 (Pin_7)
- net GPIO6: now also J30.8 (Pin_8)
- net GPIO7: now also J30.9 (Pin_9)
- net GPIO8: now also J30.10 (Pin_10)
- net GPIO9: now also J30.11 (Pin_11)
- net PWM0: now also J27.2 (Pin_2)
- net PWM1: now also J27.3 (Pin_3)
- net PWM2: now also J27.4 (Pin_4)
- net PWM3: now also J27.5 (Pin_5)
- net PWM4: now also J27.6 (Pin_6)
- net PWM5: now also J27.7 (Pin_7)
- net PWM6: now also J27.8 (Pin_8)
- net PWM7: now also J27.9 (Pin_9)
- net SPARE_P170: now also J31.2 (Pin_2)
- net SPARE_P171: now also J31.3 (Pin_3)
- net SPARE_P172: now also J31.4 (Pin_4)
- net SPARE_P173: now also J31.5 (Pin_5)
- net SPARE_P174: now also J31.6 (Pin_6)
- net SPARE_P175: now also J31.7 (Pin_7)
- net SPARE_P176: now also J31.8 (Pin_8)
- net SPARE_P177: now also J31.9 (Pin_9)
- net SPARE_P178: now also J31.10 (Pin_10)
- net SPARE_P179: now also J31.11 (Pin_11)
- net SPARE_P180: now also J31.12 (Pin_12)
- net SPARE_P181: now also J31.13 (Pin_13)
- net SPARE_P182: now also J31.14 (Pin_14)
- net SPARE_P183: now also J31.15 (Pin_15)
- net SPARE_P184: now also J31.16 (Pin_16)
- net SPARE_P185: now also J31.17 (Pin_17)
- net SPARE_P186: now also J31.18 (Pin_18)
- net SPARE_P187: now also J31.19 (Pin_19)
- net SPARE_P188: now also J31.20 (Pin_20)
- net SPARE_P189: now also J31.21 (Pin_21)
- net SPARE_P190: now also J31.22 (Pin_22)
- net SPARE_P191: now also J31.23 (Pin_23)
- net SPARE_P192: now also J31.24 (Pin_24)
- net SPARE_P193: now also J32.2 (Pin_2)
- net SPARE_P194: now also J32.3 (Pin_3)
- net SPARE_P195: now also J32.4 (Pin_4)
- net SPARE_P196: now also J32.5 (Pin_5)
- net SPARE_P197: now also J32.6 (Pin_6)
- net SPARE_P198: now also J32.7 (Pin_7)
- net SPARE_P199: now also J32.8 (Pin_8)
- net SPARE_P200: now also J32.9 (Pin_9)
- net SPARE_P201: now also J32.10 (Pin_10)
- net SPARE_P202: now also J32.11 (Pin_11)
- net SPARE_P203: now also J32.12 (Pin_12)
- net SPARE_P204: now also J32.13 (Pin_13)
- net SPARE_P205: now also J32.14 (Pin_14)
- net SPARE_P206: now also J32.15 (Pin_15)
- net SPARE_P207: now also J32.16 (Pin_16)
- net SPARE_P208: now also J32.17 (Pin_17)
- net SPARE_P209: now also J32.18 (Pin_18)
- net SPARE_P210: now also J32.19 (Pin_19)
- net SPARE_P211: now also J32.20 (Pin_20)
- net SPARE_P212: now also J32.21 (Pin_21)
- net SPARE_P213: now also J32.22 (Pin_22)
- net SPARE_P214: now also J32.23 (Pin_23)
- net SPARE_P215: now also J32.24 (Pin_24)
- net SPARE_P216: now also J32.25 (Pin_25)
- net SPARE_P217: now also J33.2 (Pin_2)
- net SPARE_P218: now also J33.3 (Pin_3)
- net SPARE_P219: now also J33.4 (Pin_4)
- net SPARE_P220: now also J33.5 (Pin_5)
- net SPARE_P221: now also J33.6 (Pin_6)
- net SPARE_P222: now also J33.7 (Pin_7)
- net SPARE_P223: now also J33.8 (Pin_8)
- net SPARE_P224: now also J33.9 (Pin_9)
- net SPARE_P225: now also J33.10 (Pin_10)
- net SPARE_P226: now also J33.11 (Pin_11)
- net SPARE_P227: now also J33.12 (Pin_12)
- net SPARE_P228: now also J33.13 (Pin_13)
- net SPARE_P229: now also J33.14 (Pin_14)
- net SPARE_P230: now also J33.15 (Pin_15)
- net SPARE_P231: now also J33.16 (Pin_16)
- net SPARE_P232: now also J33.17 (Pin_17)
- net SPARE_P233: now also J33.18 (Pin_18)
- net SPARE_P234: now also J33.19 (Pin_19)
- net SPARE_P235: now also J33.20 (Pin_20)
- net SPARE_P236: now also J33.21 (Pin_21)
- net SPARE_P237: now also J33.22 (Pin_22)
- net SPARE_P238: now also J33.23 (Pin_23)
- net SPARE_P239: now also J33.24 (Pin_24)
- net SPARE_P240: now also J33.25 (Pin_25)
- net SPARE_P241: now also J34.2 (Pin_2)
- net SPARE_P242: now also J34.3 (Pin_3)
- net SPARE_P243: now also J34.4 (Pin_4)
- net SPARE_P244: now also J34.5 (Pin_5)
- net SPARE_P245: now also J34.6 (Pin_6)
- net SPARE_P246: now also J34.7 (Pin_7)
- net SPARE_P247: now also J34.8 (Pin_8)
- net SPARE_P248: now also J34.9 (Pin_9)
- net SPARE_P249: now also J34.10 (Pin_10)
- net SPARE_P250: now also J34.11 (Pin_11)
- net SPARE_P251: now also J34.12 (Pin_12)
- net SPARE_P252: now also J34.13 (Pin_13)
- net SPARE_P253: now also J34.14 (Pin_14)
- net SPARE_P254: now also J34.15 (Pin_15)
- net SPARE_P255: now also J34.16 (Pin_16)
- net SPARE_P256: now also J34.17 (Pin_17)
- net SPARE_P257: now also J34.18 (Pin_18)
- net SPARE_P258: now also J34.19 (Pin_19)
- net SPARE_P259: now also J34.20 (Pin_20)
- net SPARE_P260: now also J34.21 (Pin_21)
- net SPARE_P261: now also J34.22 (Pin_22)
- net SPARE_P262: now also J34.23 (Pin_23)
- net SPARE_P263: now also J34.24 (Pin_24)
- net SPARE_P264: now also J34.25 (Pin_25)
- net SPARE_P265: now also J35.2 (Pin_2)
- net SPARE_P266: now also J35.3 (Pin_3)
- net SPARE_P267: now also J35.4 (Pin_4)
- net SPARE_P268: now also J35.5 (Pin_5)
- net SPARE_P269: now also J35.6 (Pin_6)
- net SPARE_P270: now also J35.7 (Pin_7)
- net SPARE_P271: now also J35.8 (Pin_8)
- net SPARE_P272: now also J35.9 (Pin_9)
- net SPARE_P273: now also J35.10 (Pin_10)
- net SPARE_P274: now also J35.11 (Pin_11)
- net SPARE_P275: now also J35.12 (Pin_12)
- net SPARE_P276: now also J35.13 (Pin_13)
- net SPARE_P277: now also J35.14 (Pin_14)
- net SPARE_P278: now also J35.15 (Pin_15)
- net SPARE_P279: now also J35.16 (Pin_16)
- net SPARE_P280: now also J35.17 (Pin_17)
- net SPARE_P281: now also J35.18 (Pin_18)
- net SPARE_P282: now also J35.19 (Pin_19)
- net SPARE_P283: now also J35.20 (Pin_20)
- net SPARE_P284: now also J35.21 (Pin_21)
- net SPARE_P285: now also J35.22 (Pin_22)
- net SPARE_P286: now also J35.23 (Pin_23)
- net SPARE_P287: now also J35.24 (Pin_24)
- net SPARE_P288: now also J35.25 (Pin_25)
- net SSI0_CE0: now also J25.5 (Pin_5)
- net SSI0_CE1: now also J25.6 (Pin_6)
- net SSI0_CLK: now also J25.2 (Pin_2)
- net SSI0_DR: now also J25.4 (Pin_4)
- net SSI0_DT: now also J25.3 (Pin_3)
- net SSI0_GPC: now also J25.7 (Pin_7)
