File: hw/teacup-carrier.kicad_pcb (KiCad board)
At the start: 4 copper layers, 280 x 240 mm, 128 parts, among them J1 AH58893-T9B10-3F, J2 TYPE-C-31-M-12, J20 HDR_J20, J21 HDR_J21, J22 HDR_J22, J23 HDR_J23, J24 HDR_J24, J25 HDR_J25, J26 HDR_J26, J27 HDR_J27, J28 HDR_J28, J29 HDR_J29, J3 TE_292303-7, J30 HDR_J30, J31 HDR_J31, J32 HDR_J32, J33 HDR_J33, J34 HDR_J34, J35 HDR_J35, J4 Hirose_DM3D-SF, J5 Wuerth_694106301002, J6 AudioJack4_Ground, J7 SFW15R-2STE1LF, J8 SFW15R-2STE1LF, J9 TYPE-C-31-M-12, Q1 AO3401A, Q2 AO3401A, SW1 SSSS711403, SW2 SSSS711403, U1 AP62600SJ-7, U10 TS5A3166, U11 DIP-8 Socket, U12 TPS2053BDR, U13 W25Q32JVSS, U14 TPS22990DMLR, U15 TCA9555PWR, U2 AP62300WU-7, U3 MCP4661-104E_ST, U4 TPS22990DMLR, U5 AZ1117CH-3.3TRG1, U6 AZ1117CH-1.8TRG1, U7 AP62300WU-7, U8 ESP32-S3-WROOM-1-N16R2, U9 TS5A3166

Commit message: Convert large pin-breakout headers to double-row, J1-ordered pinout
J20/J21/J25/J27/J30-J35 now use Conn_02xNN_Odd_Even + PinHeader_2xNN
footprints instead of single-row 1xNN -- half the physical length, and
KiCad's odd/even pin numbering keeps each header's signals in the same
J1-sequential order they were already assigned, just zig-zagged across
two columns instead of one long row. Odd GND+signal counts get a 2nd
GND appended at the far pin to fill the row evenly. J22-J24/J26/J28/J29
(<=5 pins) stay single-row.

Regenerated headers.kicad_sch/teacup-carrier.kicad_sch/CONNECTIONS.txt
via the existing schgen toolchain: 0 overlaps, ERC violation set
unchanged from baseline (429, byte-identical). Rebuilt
teacup-carrier.kicad_pcb via build_pcb.py for the new footprints --
rough cluster placement only, no routing.
Parts:
- C13, C23: value 1nF_TBD -> 1nF
- J20, J21: footprint PinHeader_1x11_P2.54mm_Vertical -> PinHeader_2x06_P2.54mm_Vertical
- J25: footprint PinHeader_1x07_P2.54mm_Vertical -> PinHeader_2x04_P2.54mm_Vertical
- J27: footprint PinHeader_1x09_P2.54mm_Vertical -> PinHeader_2x05_P2.54mm_Vertical
- J30: footprint PinHeader_1x17_P2.54mm_Vertical -> PinHeader_2x09_P2.54mm_Vertical
- J31: footprint PinHeader_1x24_P2.54mm_Vertical -> PinHeader_2x12_P2.54mm_Vertical
- J32, J33, J34, J35: footprint PinHeader_1x25_P2.54mm_Vertical -> PinHeader_2x13_P2.54mm_Vertical
- moved J1 185.5 mm to (155.4, 40.1)
- moved J35 174.8 mm to (223.8, 23.3)
- moved L3 174.1 mm to (118.3, 178.3)
- moved J28 169.8 mm to (59.9, 47.8)
- moved JP5 169.7 mm to (36.3, 182.4)
- moved R27 160.4 mm to (30.3, 166.7)
- moved U8 160.3 mm to (45.1, 119.2)
- moved U13 158.6 mm to (62.1, 123.2)
- moved R36 155.4 mm to (40.3, 161.7)
- moved J34 155.1 mm to (188.3, 23.3)
- moved R28 151.4 mm to (39.3, 168.7)
- moved J30 151.1 mm to (59.8, 23.3)
- moved R37 150.5 mm to (37.3, 164.7)
- moved J8 145.2 mm to (146.9, 69.7)
- moved C1 145.2 mm to (110.3, 119.3)
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