File: hw/.history/teacup-carrier.kicad_sch (KiCad schematic)
At the start: 59 parts, among them J1 AH58893-T9B10-3F, J2 TYPE-C-31-M-12, J3 TE_292303-7, J4 Hirose_DM3D-SF, J5 Wuerth_694106301002, J6 AudioJack4_Ground, J7 SFW15R-2STE1LF, J8 SFW15R-2STE1LF, SW1 SSSS711403, U1 AP62600SJ-7, U10 TS5A3166, U11 DIP-8 Socket, U12 TPS2053BDR, U2 AP62300WU-7, U3 MCP4661-104E_ST, U4 TPS22990DMLR, U5 AZ1117CH-3.3TRG1, U6 AZ1117CH-1.8TRG1, U7 AP62300WU-7, U8 ESP32-S3-WROOM-1-N16R2, U9 TS5A3166

Commit message: Carrier board: BMC power isolation, ESP-Hosted link, GPIO expander
Rebuilds the schematic to connectivity-by-label per BUILD.md (zero
wires/junctions) across all four sections, and adds the BMC power
architecture, connector crossings, and safety fixes worked out this
session:

- Dedicated BMC USB-C (J9), isolated 5V domains (+5V_BMC/+5V_ALT/+5V_SW),
  priority DC-jack-over-USB-C P-FET OR (Q1/Q2), 2:1 load-switch select
  (U4/U14) with a genuine ON-OFF-ON manual override (SW2)
- D1/D2 diode-OR so the BMC stays powered on ALT-only input without
  reopening the J9 backfeed path
- JP1 provisioning jumper + mandatory bring-up checklist: gates SW2 until
  the digipot's NV memory has been confirmed safe, closing the
  factory-mid-scale-default overvoltage gap on VCORE
- GPIO expander (U15, TCA9555PWR) frees 9 ESP32 GPIOs for a full-duplex
  SPI link to the interposer SoC (ESP-Hosted WiFi/BLE co-processor),
  while keeping flash chip-select and power-domain switching native for
  margin testing
- microSD, headphone jack, and both MIPI camera FFCs now cross the DDR4
  connector to the interposer, with GND isolation around each block
- J2/J3 share one USB host data pair to the interposer (peripheral use,
  independent of J2's power role)
- Added missing primary SOIC-8 NOR flash chip (W25Q32JVSS) to match the
  reference board's dual-NOR layout

docs/UNIVERSAL.md updated throughout to match; CONNECTIONS.txt and the
ESP32 pinout reference regenerated from the current netlist.
Parts:
- added C23: 1nF_TBD, Capacitor_SMD:C_0402_1005Metric, symbol Device:C
- added D1, D2: PMEG2010ER, Diode_SMD:D_SOD-123W, symbol Device:D_Schottky
- added J9: TYPE-C-31-M-12, Connector_USB:USB_C_Receptacle_HRO_TYPE-C-31-M-12, symbol Connector:USB_C_Receptacle_USB2.0_16P
- added JP1: PROVISIONED, Connector_PinHeader_2.54mm:PinHeader_1x02_P2.54mm_Vertical, symbol Connector_Generic:Conn_01x02
- added Q1, Q2: AO3401A, Package_TO_SOT_SMD:SOT-23, symbol Device:Q_PMOS
- added R15, R17, R20, R22: 100k, Resistor_SMD:R_0402_1005Metric, symbol Device:R
- added R16: 4.7k, Resistor_SMD:R_0402_1005Metric, symbol Device:R
- added R18, R19: 5.1k, Resistor_SMD:R_0402_1005Metric, symbol Device:R
- added R21, R23: 1k, Resistor_SMD:R_0402_1005Metric, symbol Device:R
- added R24: 10k, Resistor_SMD:R_0402_1005Metric, symbol Device:R
- added SW2: SSSS711403, teacup-carrier:SW-TH_SSSS711403, symbol teacup-carrier:SSSS711403
- added U13: W25Q32JVSS, Package_SO:SOIC-8_5.23x5.23mm_P1.27mm, symbol teacup-carrier:W25Q32JVSS
- added U14: TPS22990DMLR, teacup-carrier:WSON-10_L3.0-W2.0-P0.50-BL-EP_TI_DML, symbol teacup-carrier:TPS22990DMLR
- added U15: TCA9555PWR, Package_SO:TSSOP-24_4.4x7.8mm_P0.65mm, symbol teacup-carrier:TCA9555PWR
Connections:
- net RESERVED_P41 is gone; now on net USBA_HOST_DP: J1.41 (P41)
- net RESERVED_P42 is gone; now on net USBA_HOST_DM: J1.42 (P42)
- net RESERVED_P48 is gone; now on net HOSTED_DATA_READY: J1.48 (P48)
- net +3V3: now also C19.1, L3.2, R24.1, U13.8 (VCC), U15.24 (VCC); no longer C17.2
- net +3V3_ALWAYS: now also C21.1; no longer C21.2
- net +5V_SW: now also C1.1, C16.1, C2.1, C6.1, R1.1, U14.10 (VOUT), U14.8 (VOUT), U14.9 (VOUT); no longer R1.2, U1.3 (EN)
- net BMC_USB_DM: now also J9.A7 (D-), J9.B7 (D-); no longer J2.A7 (D-), J2.B7 (D-)
- net BMC_USB_DP: now also J9.A6 (D+), J9.B6 (D+); no longer J2.A6 (D+), J2.B6 (D+)
- net DCJACK_PRESENT: now also U15.13 (P10)
- net GND: now also C21.2, C4.2, J1.12 (P12), J1.20 (P20), J1.21 (P21), J1.22 (P22), J1.36 (P36), J1.37 (P37), J1.38 (P38), J1.39 (P39), J1.40 (P40), J1.49 (P49), J1.51 (P51), J1.57 (P57), J1.59 (P59), J1.6 (P6), J1.63 (P63), J1.66 (P66), J1.69 (P69), J1.7 (P7), J1.72 (P72), J1.76 (P76), J1.79 (P79), J1.8 (P8), J1.82 (P82), J1.85 (P85), U1.5 (FSEL), U3.12 (A2), U3.5 (P1B), C23.2, J9.A1 (GND), J9.A12 (GND), J9.B1 (GND), J9.B12 (GND), J9.S1 (SHIELD), R15.2, R17.2, R18.2, R19.2, R20.2, R22.2, U13.4 (GND), U14.6 (GND), U15.12 (GND), U15.2 (A1), U15.21 (A0), U15.3 (A2); no longer C21.1, C4.1
- net HPOUTL: now also J1.58 (P58)
- net I2C_PWR_SCL: now also U15.22 (SCL)
- net I2C_PWR_SDA: now also U15.23 (SDA)
- net MIPI0_CLKN: now also J1.70 (P70)
- net MIPI0_CLKP: now also J1.71 (P71)
- net MIPI0_D0N: now also J1.64 (P64)
- net MIPI0_D0P: now also J1.65 (P65)
- net MIPI0_D1N: now also J1.67 (P67)
- net MIPI0_D1P: now also J1.68 (P68)
- net MIPI0_GPIO: now also J1.60 (P60)
- net MIPI0_SCCB_SCL: now also J1.62 (P62)
- net MIPI0_SCCB_SDA: now also J1.61 (P61)
- net MIPI1_CLKN: now also J1.83 (P83)
- net MIPI1_CLKP: now also J1.84 (P84)
- net MIPI1_D0N: now also J1.77 (P77)
- net MIPI1_D0P: now also J1.78 (P78)
- net MIPI1_D1N: now also J1.80 (P80)
- net MIPI1_D1P: now also J1.81 (P81)
- net MIPI1_GPIO: now also J1.73 (P73)
- net MIPI1_SCCB_SCL: now also J1.75 (P75)
- net MIPI1_SCCB_SDA: now also J1.74 (P74)
- net MSC0_CLK: now also J1.50 (P50)
- net MSC0_CMD: now also J1.52 (P52)
- net MSC0_D0: now also J1.53 (P53)
- net MSC0_D1: now also J1.54 (P54)
- net MSC0_D2: now also J1.55 (P55)
- net MSC0_D3_CD: now also J1.56 (P56)
- net NOR_U4_CE: now also U13.1 (~{CS})
- net PG_SW5V: now also U15.7 (P03); no longer U8.23 (GPIO21)
- net PG_VCORE: now also U15.8 (P04); no longer U8.24 (GPIO47)
- net SFC_CLK: now also U13.6 (CLK)
- net SFC_IO0: now also U13.5 (DI(IO0))
- net SFC_IO1: now also U13.2 (DO(IO1))
- net SFC_IO2: now also U13.3 (IO2)
- net SFC_IO3: now also U13.7 (IO3)
- net SW_SENSE_1: now also R10.2, U15.10 (P06); no longer U8.28 (SPIIO6)
- net SW_SENSE_4: now also R11.2, U15.11 (P07); no longer U8.29 (SPIIO7)
- net USBA_HOST_DM: now also J2.A7 (D-), J2.B7 (D-)
- net USBA_HOST_DP: now also J2.A6 (D+), J2.B6 (D+)
- net USB_EN1: now also U15.4 (P00); no longer U8.8 (GPIO15)
- net USB_EN2: now also U15.5 (P01); no longer U8.9 (GPIO16)
- net USB_EN3: now also U15.6 (P02); no longer U8.25 (GPIO48)
- net VCORE: now also C9.1
- net VDDR: now also C11.1, L2.2; no longer C7.2
- net U1_SW: now reaches L1.1
- net U1_SW: now also C3.2, U1.8 (SW)
- net U4_CT: now reaches C13.1, U4.1 (CT)
- net +5V_BMC: now reaches U4.4 (VBIAS)
- net +5V_BMC: now also U4.11 (VIN), U4.3 (VIN), D1.2 (A), J9.A4 (VBUS), J9.A9 (VBUS), J9.B4 (VBUS), J9.B9 (VBUS)
- net USBC_CC1: now reaches J2.A5 (CC1), R12.1
- net U1_SS: now reaches C5.1, U1.10 (SS/TR)
- net U1_BST: now reaches C3.1, U1.7 (BST)
- net P3V3_FB: now reaches R6.2, R7.1
- net P3V3_FB: now also U7.4 (FB)
- net USBC_CC2: now reaches J2.B5 (CC2), R13.1
- net U7_BST: now reaches C17.1, U7.6 (BST)
- net U2_EN: now reaches R3.2
- net U2_EN: now also U2.5 (EN)
- net U2_SW: now reaches U2.2 (SW)
- net U2_SW: now also C7.2, L2.1
- net U2_BST: now reaches C7.1, U2.6 (BST)
- net U7_EN: now reaches R5.2
- net U7_EN: now also U7.5 (EN)
- net U1_VCC: now reaches U1.9 (VCC)
- net U1_VCC: now also C4.1
- net U5_VIN: now reaches C14.1
- net U5_VIN: now also U5.1 (IN), D1.1 (K), D2.1 (K)
- net U7_SW: now reaches U7.2 (SW)
- net U7_SW: now also C17.2, L3.1
- net HOSTED_RESET: now reaches J1.86 (P86)
- net HOSTED_RESET: now also R8.2, U8.3 (EN)
- net RESERVED_P87: now reaches J1.87 (P87)
- net RESERVED_P88: now reaches J1.88 (P88)
- net RESERVED_P89: now reaches J1.89 (P89)
- net RESERVED_P90: now reaches J1.90 (P90)
- net RESERVED_P91: now reaches J1.91 (P91)
- net RESERVED_P92: now reaches J1.92 (P92)
- net RESERVED_P93: now reaches J1.93 (P93)
- net RESERVED_P94: now reaches J1.94 (P94)
- net RESERVED_P95: now reaches J1.95 (P95)
- net RESERVED_P96: now reaches J1.96 (P96)
- net U8_BOOT: now reaches R9.2, U8.27 (GPIO0)
- net SW5V_EN_ALT: now reaches U8.16 (GPIO46)
- net SW5V_EN_ALT: now also R23.1
- net HOSTED_DATA_READY: now reaches U8.26 (GPIO45)
- net +5V_IN renamed ALTUSB_VBUS
- net ALTUSB_VBUS: now also Q2.S; no longer J5.1, U4.11 (VIN), U4.3 (VIN), U5.1 (IN)
- net RESERVED_P43 renamed HOSTED_SPI_CLK
- net HOSTED_SPI_CLK: now also U8.8 (GPIO15)
- net RESERVED_P44 renamed HOSTED_SPI_MOSI
- net HOSTED_SPI_MOSI: now also U8.9 (GPIO16)
- net RESERVED_P45 renamed HOSTED_SPI_MISO
- net HOSTED_SPI_MISO: now also U8.23 (GPIO21)
- net RESERVED_P46 renamed HOSTED_SPI_CS
- net HOSTED_SPI_CS: now also U8.24 (GPIO47)
- net RESERVED_P47 renamed HOSTED_HANDSHAKE
- net HOSTED_HANDSHAKE: now also U8.25 (GPIO48)
- net SW5V_EN renamed EN_SW_BMC
- net EN_SW_BMC: now also R20.1, R21.2, SW2.1; no longer U8.38 (GPIO2)
- new net +5V_ALT: D2.2 (A), JP1.1 (Pin_1), Q1.D, Q2.D, U14.11 (VIN), U14.3 (VIN), U14.4 (VBIAS)
- new net DCJACK_VBUS: J5.1, Q1.S, R16.1
- new net EN_SW_ALT: R22.1, R23.2, SW2.4, U14.5 (ON)
- new net EXP_INT: U15.1 (~{INT}), U8.28 (SPIIO6)
- new net PG_SW5V_ALT: R24.2, U14.7 (PG), U15.9 (P05)
- new net Q1_GATE: Q1.G, R15.1
- new net Q2_GATE: Q2.G, R16.2, R17.1
- new net SW2_POLE: JP1.2 (Pin_2), SW2.3
- new net SW5V_EN_BMC: R21.1, U8.38 (GPIO2)
- new net U14_CT: C23.1, U14.1 (CT)
- new net U1_EN: R1.2, U1.3 (EN)
- new net USBC2_CC1: J9.A5 (CC1), R18.1
- new net USBC2_CC2: J9.B5 (CC2), R19.1
